File: PC9821 26 pin floppy adapter.sch (KiCad schematic (older format))
At the start: 3 parts

Commit message: Final version of the panel mount 26-pin version - 1
Parts:
- PC98-F1: footprint Connector_IDC:IDC-Header_2x13_P2.54mm_Horizontal -> Connector_IDC:IDC-Header_2x13_P2.54mm_Vertical
Changed lines of the file:
@@
 F 0 "PC98-F1" H 3475 4767 50  0000 C CNN
 F 1 "Male 26-pin from floppy cable" H 3475 4676 50  0000 C CNN
-F 2 "Connector_IDC:IDC-Header_2x13_P2.54mm_Horizontal" H 3425 3950 50  0001 C CNN
+F 2 "Connector_IDC:IDC-Header_2x13_P2.54mm_Vertical" H 3425 3950 50  0001 C CNN
 F 3 "~" H 3425 3950 50  0001 C CNN
 	1    3425 3950

Commit message: Final version that I just sent off to Osh
Parts:
- PC98-F1: footprint Connector_IDC:IDC-Header_2x13_P2.54mm_Vertical -> Connector_IDC:IDC-Header_2x13_P2.54mm_Horizontal
Changed lines of the file:
@@
 F 0 "PC98-F1" H 3475 4767 50  0000 C CNN
 F 1 "Male 26-pin from floppy cable" H 3475 4676 50  0000 C CNN
-F 2 "Connector_IDC:IDC-Header_2x13_P2.54mm_Vertical" H 3425 3950 50  0001 C CNN
+F 2 "Connector_IDC:IDC-Header_2x13_P2.54mm_Horizontal" H 3425 3950 50  0001 C CNN
 F 3 "~" H 3425 3950 50  0001 C CNN
 	1    3425 3950

Commit message: v1.1, a huge ridiculous board that doesn't have a molex power connector on it anymore
Parts:
- removed POWER1: 4 pin male molex power, XESS connector lib:xess-MOLEX-8981-04P, symbol Connector:Conn_01x04_Male
Connections:
- net labels added: +5V_1, +5V_2, +5V_3
- net labels removed: +12V, +5V
- wire segments 142 -> 133
- no-connect marks 4 -> 3
Changed lines of the file:
@@
 	1    0    0    -1
 $EndComp
-$Comp
-L Connector:Conn_01x04_Male POWER1
-U 1 1 5B7C4158
-P 3775 5350
-F 0 "POWER1" H 3881 5628 50  0000 C CNN
-F 1 "4 pin male molex power" H 3881 5537 50  0000 C CNN
-F 2 "XESS connector lib:xess-MOLEX-8981-04P" H 3775 5350 50  0001 C CNN
-F 3 "~" H 3775 5350 50  0001 C CNN
-	1    3775 5350
-	1    0    0    -1
-$EndComp
-Text Label 3975 5250 0    50   ~ 0
-+12V
-Text Label 3975 5350 0    50   ~ 0
-GND
-Text Label 3975 5450 0    50   ~ 0
-GND
-Text Label 3975 5550 0    50   ~ 0
-+5V
 Text Label 3225 3350 2    50   ~ 0
-+5V
-Wire Wire Line
-	3225 3350 1225 3350
-Wire Wire Line
-	1225 3350 1225 3450
-Wire Wire Line
-	1225 7225 3975 7225
-Wire Wire Line
-	3975 7225 3975 5550
++5V_1
 Text Label 3225 3450 2    50   ~ 0
-+5V
-Wire Wire Line
-	3225 3450 1225 3450
-Connection ~ 1225 3450
-Wire Wire Line
-	1225 3450 1225 3550
++5V_2
 Text Label 3225 3550 2    50   ~ 0
-+5V
-Wire Wire Line
-	3225 3550 1225 3550
-Connection ~ 1225 3550
-Wire Wire Line
-	1225 3550 1225 7225
++5V_3
 Text Label 3225 3950 2    50   ~ 0
 GND
@@
 	8225 2525 8225 5450
 Wire Wire Line
-	3975 5450 4750 5450
-Connection ~ 4750 5450
-Wire Wire Line
 	4750 5450 8225 5450
 Text Label 6725 3450 2    50   ~ 0
@@
 	2075 3750 3225 3750
 Wire Wire Line
-	7225 3650 8075 3650
-Wire Wire Line
-	8075 3650 8075 5300
-Wire Wire Line
-	2125 5300 2125 3650
-Wire Wire Line
-	2125 3650 3225 3650
-Wire Wire Line
-	2125 5300 8075 5300
-Wire Wire Line
 	7225 3450 8075 3450
 Wire Wire Line
@@
 NoConn ~ 7225 3750
 NoConn ~ 7225 3350
-NoConn ~ 3975 5250
 Wire Wire Line
 	6725 3150 6725 2125
@@
 Wire Wire Line
 	2375 4050 1950 4050
+Wire Wire Line
+	3225 3650 2550 3650
+Wire Wire Line
+	2550 3650 2550 5850
+Wire Wire Line
+	2550 5850 7925 5850
+Wire Wire Line
+	7925 5850 7925 3650
+Wire Wire Line
+	7925 3650 7225 3650
 $EndSCHEMATC

Commit message: A revision with a Molex 8981 power connector to provide power OUT to the 34-pin floppy drive
Parts:
- added PWR1: Molex 8981 Power Out, XESS connector lib:xess-MOLEX-8981-04P, symbol Connector_Generic:Conn_01x04
Connections:
- net labels added: +5V_OUT
- wire segments 133 -> 141
- no-connect marks 3 -> 4
Changed lines of the file:
@@
 	1950 3950 1950 4050
 Wire Wire Line
-	1950 4725 4750 4725
+	1950 4725 2675 4725
 Wire Wire Line
 	4750 4725 4750 5450
@@
 Wire Wire Line
 	7925 3650 7225 3650
+$Comp
+L Connector_Generic:Conn_01x04 PWR1
+U 1 1 5B89CFB2
+P 3925 5325
+F 0 "PWR1" H 4004 5317 50  0000 L CNN
+F 1 "Molex 8981 Power Out" H 4004 5226 50  0000 L CNN
+F 2 "XESS connector lib:xess-MOLEX-8981-04P" H 3925 5325 50  0001 C CNN
+F 3 "~" H 3925 5325 50  0001 C CNN
+	1    3925 5325
+	1    0    0    -1
+$EndComp
+Text Label 3725 5325 2    50   ~ 0
+GND
+Text Label 3725 5425 2    50   ~ 0
+GND
+Text Label 3725 5525 2    50   ~ 0
++5V_OUT
+NoConn ~ 3725 5225
+Wire Wire Line
+	3725 5325 2675 5325
+Connection ~ 2675 4725
+Wire Wire Line
+	2675 4725 4750 4725
+Wire Wire Line
+	3725 5425 2675 5425
+Wire Wire Line
+	2675 4725 2675 5325
+Connection ~ 2675 5325
+Wire Wire Line
+	2675 5325 2675 5425
+Wire Wire Line
+	3725 5525 1675 5525
+Wire Wire Line
+	1675 5525 1675 3350
+Wire Wire Line
+	1675 3350 3225 3350
 $EndSCHEMATC

Commit message: Revision 1.4 - has bigger holes for the Molex connector, and the Molex connector is on the other side
Parts:
- PWR1: footprint XESS connector lib:xess-MOLEX-8981-04P -> 7709971:770997-1
Changed lines of the file:
@@
 EESchema Schematic File Version 4
+LIBS:PC9821 26 pin floppy adapter-cache
 EELAYER 26 0
 EELAYER END
@@
 F 0 "PWR1" H 4004 5317 50  0000 L CNN
 F 1 "Molex 8981 Power Out" H 4004 5226 50  0000 L CNN
-F 2 "XESS connector lib:xess-MOLEX-8981-04P" H 3925 5325 50  0001 C CNN
+F 2 "7709971:770997-1" H 3925 5325 50  0001 C CNN
 F 3 "~" H 3925 5325 50  0001 C CNN
 	1    3925 5325

Commit message: v1.5 revision
Parts:
- added JP1: 300/360 control, Jumper:SolderJumper-2_P1.3mm_Bridged2Bar_RoundedPad1.0x1.5mm, symbol Device:Jumper_NC_Small
Connections:
- wire segments 141 -> 146
Changed lines of the file:
@@
 EESchema Schematic File Version 4
-LIBS:PC9821 26 pin floppy adapter-cache
-EELAYER 26 0
+EELAYER 30 0
 EELAYER END
 $Descr A4 11693 8268
@@
 	6725 3150 6725 2125
 Wire Wire Line
-	6725 2125 2375 2125
-Wire Wire Line
 	2375 2125 2375 4050
 Connection ~ 2375 4050
@@
 	3725 5525 1675 5525
 Wire Wire Line
-	1675 5525 1675 3350
+	1675 5525 1675 3550
 Wire Wire Line
 	1675 3350 3225 3350
+Text Label 6025 2525 0    50   ~ 0
+GND
+$Comp
+L Device:Jumper_NC_Small JP1
+U 1 1 61F57564
+P 6475 2125
+F 0 "JP1" H 6475 2337 50  0000 C CNN
+F 1 "300/360 control" H 6475 2246 50  0000 C CNN
+F 2 "Jumper:SolderJumper-2_P1.3mm_Bridged2Bar_RoundedPad1.0x1.5mm" H 6475 2125 50  0001 C CNN
+F 3 "~" H 6475 2125 50  0001 C CNN
+	1    6475 2125
+	1    0    0    -1
+$EndComp
+Wire Wire Line
+	6725 2125 6575 2125
+Wire Wire Line
+	6375 2125 2375 2125
+Wire Wire Line
+	3225 3450 1675 3450
+Connection ~ 1675 3450
+Wire Wire Line
+	1675 3450 1675 3350
+Wire Wire Line
+	3225 3550 1675 3550
+Connection ~ 1675 3550
+Wire Wire Line
+	1675 3550 1675 3450
 $EndSCHEMATC

Commit message: V2.0: Floppy cable variant to support two drives
Parts:
- GOTEK1: value 34-pin female IDC to Gotek -> 34-pin female IDC to standard PC floppy cable; footprint Connector_IDC:IDC-Header_2x17_P2.54mm_Horizontal -> Connector_IDC:IDC-Header_2x17_P2.54mm_Vertical
Changed lines of the file:
@@
 P 6925 3950
 F 0 "GOTEK1" H 6975 4967 50  0000 C CNN
-F 1 "34-pin female IDC to Gotek" H 6975 4876 50  0000 C CNN
-F 2 "Connector_IDC:IDC-Header_2x17_P2.54mm_Horizontal" H 6925 3950 50  0001 C CNN
+F 1 "34-pin female IDC to standard PC floppy cable" H 6975 4876 50  0000 C CNN
+F 2 "Connector_IDC:IDC-Header_2x17_P2.54mm_Vertical" H 6925 3950 50  0001 C CNN
 F 3 "~" H 6925 3950 50  0001 C CNN
 	1    6925 3950
